Commit message: CAD visual meshes in RViz (cosmetic, kinematics untouched)
Co-Authored-By: Claude Sonnet 5 <noreply@anthropic.com>

File: src/scara_description/urdf/scara.urdf (robot description, URDF)
Before this commit: robot scara, 8 links, 7 joints
Links:
- link base_link: geometry collision cylinder length=0.40 radius=0.07; visual mesh filename=package://scara_description/meshes/base_column.stl scale=0.001 0.001 0.001
- link link1: geometry collision box size=0.28 0.07 0.055; visual mesh filename=package://scara_description/meshes/upper_arm.stl scale=0.001 0.001 0.001
- link link2: geometry collision box size=0.23 0.055 0.045; visual mesh filename=package://scara_description/meshes/forearm.stl scale=0.001 0.001 0.001
- link link3: geometry collision cylinder length=0.10 radius=0.016; visual mesh filename=package://scara_description/meshes/quill.stl scale=0.001 0.001 0.001
- link link4: geometry collision cylinder length=0.03 radius=0.022; visual mesh filename=package://scara_description/meshes/spindle_tip.stl scale=0.001 0.001 0.001
